File: sensor16ADC/sensr-circuit/sensr-circuit.kicad_pcb (KiCad board)
At the start: 2 copper layers, 20 parts, among them J1 Conn_01x09_Male, U1 WeMos_D1_mini, U2 CD74HC4067M, U3 AMS1117CD-1.5

Commit message: circuit with 24V to 3.3V regulator
Parts:
- U3: value AMS1117CD-1.5 -> Pololu-D24V3F3; footprint AudioChannel:AMS1117 -> AudioChannel:Pololu-D24V3F3
- moved U3 10.5 mm to (45.2, 41.8), turned to 90 degrees
Connections:
- U3 pad 1: GND -> +24V
- U3 pad 2: 3.3V -> +24V
- U3 pad 3: +6.4V -> GND
Routing:
- net +24V: track 10.2 -> 85.6 mm, vias 0 -> 3
- net +6.4V: track 66.4 -> 14.6 mm
- net 3.3V: track 85.7 -> 95.7 mm

Commit message: circuit fix
Parts:
- added C1: 33uF, Capacitor_THT:CP_Radial_D5.0mm_P2.50mm, F.Cu at (43.0, 44.5)
- R1, R10, R11, R12, R13, R14, R15, R16, R2, R3, R4, R5, R6, R7, R8, R9: footprint Resistor_THT:R_Axial_DIN0204_L3.6mm_D1.6mm_P1.90mm_Vertical -> Resistor_THT:R_Axial_DIN0204_L3.6mm_D1.6mm_P7.62mm_Horizontal
- moved R10 30.0 mm to (67.0, 55.0), turned to 0 degrees
- moved R14 30.0 mm to (67.0, 60.0), turned to 0 degrees
- moved R16 30.0 mm to (67.0, 62.5), turned to 0 degrees
- moved R8 30.0 mm to (67.0, 52.5), turned to 0 degrees
- moved R2 29.9 mm to (67.0, 45.0), turned to 0 degrees
- moved R4 29.9 mm to (67.0, 47.5), turned to 0 degrees
- moved R6 29.9 mm to (67.0, 50.0), turned to 0 degrees
- moved R12 29.8 mm to (67.1, 57.5), turned to 0 degrees
- moved R15 3.10 mm to (88.0, 62.5)
- moved R3 3.02 mm to (88.0, 47.6)
- moved R1 3.02 mm to (88.0, 45.0)
- moved R11 3.00 mm to (88.0, 57.5)
- moved R13 3.00 mm to (88.0, 60.0)
- moved R5 3.00 mm to (88.0, 50.0)
- moved R7 3.00 mm to (88.0, 52.5)
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Connections:
- R10 pad 2: +16.2V -> Net-(R10-Pad2)
- R12 pad 2: +19.4V -> Net-(R11-Pad2)
- R14 pad 2: +22.6 -> Net-(R13-Pad2)
- R16 pad 2: +24V -> Net-(R15-Pad2)
- R2 pad 2: +3.2V -> Net-(R1-Pad2)
- R4 pad 2: +6.4V -> Net-(R3-Pad2)
- R6 pad 2: +9.6V -> Net-(R5-Pad2)
- R8 pad 2: +12.8V -> Net-(R7-Pad2)
- R9 pad 2: Net-(R9-Pad2) -> Net-(R10-Pad2)
- U2 pad 5: Net-(R9-Pad2) -> Net-(R10-Pad2)
Routing:
- net +24V: track 85.6 -> 100.1 mm
- net +3.2V: track 14.6 -> 3.79 mm
- net +6.4V: track 14.6 -> 3.81 mm
- net GND: track 135.7 -> 126.5 mm
- net +12.8V: track 10.2 -> 3.76 mm
- net +16.2V: track 10.2 -> 3.76 mm
- net +9.6V: track 10.2 -> 3.77 mm
- net +22.6: track 10.1 -> 3.79 mm
- net +19.4V: track 10.1 -> 3.77 mm
- net Net-(R10-Pad2): track 0.00 -> 5.76 mm
- net Net-(R9-Pad2): track 5.60 -> 0.00 mm
Other:
- board text added: "CD74HC4067M"
- board text added: "D1 Mini"

Commit message: bat-mon-firmware:0.5.0 Temperature sensor DS18B20
Parts:
- added J2: Conn_01x03_Male, Connector_JST:JST_EH_B3B-EH-A_1x03_P2.50mm_Vertical, F.Cu at (57.6, 88.6)
- added R17: 3k9, Resistor_THT:R_Axial_DIN0309_L9.0mm_D3.2mm_P2.54mm_Vertical, F.Cu at (50.8, 88.6)
Connections:
- U1 pad 6: Net-(U1-Pad6) -> 1Wire
Routing:
- net 1Wire: track 0.00 -> 43.9 mm, vias 0 -> 2
- net 3.3V: track 95.7 -> 137.2 mm, vias 4 -> 6
- net GND: track 126.5 -> 148.5 mm, vias 6 -> 8
